Commit message: feat(robot-control): add WASD keyboard control for robot manipulation
Add new WASD keyboard control component with support for WQSD/ZXCV/1234 key mappings to control robot joints. Includes interactive button panel with visual feedback and continuous movement support. The control panel can be toggled and positioned on screen.

Also includes minor adjustment to URDF joint limit for better movement range.

File: public/URDFs/so101.urdf (robot description, URDF)
Before this commit: robot so100, 10 links, 9 joints
Joints:
- joint Pitch: limit lower=1.39467 upper=4.88692 effort=10 velocity=10 -> lower=1.39626 upper=4.88692 effort=10 velocity=10
